File: osvetlenie/osvetlenie.kicad_sch (KiCad schematic)
At the start: 66 parts, among them IC1 TJA1040T_CM,118, J1 LED_CHIP3_OUT, J2 LED_CHIP4_OUT, J3 LED_CHIP1_OUT, J4 LED_CHIP2_OUT, J5 Jack-DC-48V, J6 CAN_bus, J7 LIGHT_BULB_OUT, J8 LED_STRIP, K1 RZ03-1C4-D005, K2 RZ03-1C4-D005, K3 RZ03-1C4-D005, K4 LDD-700H, K5 LDD-700H, K6 LDD-700H, K7 LDD-700H, Q1 BC847, Q2 BC847, Q3 BC847, SW1 SW_MEC_5G, SW2 SW_MEC_5G, U1 ESP32-WROOM-32D, U2 LM2596S-12/ADJ, U3 LM2596S-5/ADJ, U4 LM1117-1.8

Commit message: Added PCB
Parts:
- removed C5: 0.1u, Capacitor_SMD:C_0603_1608Metric, symbol Device:C
- removed SW1, SW2: SW_MEC_5G, Button_Switch_SMD:SW_SPST_EVQPE1, symbol Switch:SW_MEC_5G
- removed U4: LM1117-1.8, symbol Regulator_Linear:LM1117-1.8
- added C17: 4u7, Capacitor_SMD:C_0603_1608Metric, symbol Device:C_Small
- added C18: 22u, Capacitor_Tantalum_SMD:CP_EIA-3216-18_Kemet-A, symbol Device:C_Polarized
- added C5: 0u1, Capacitor_SMD:C_0603_1608Metric, symbol Device:C_Small
- added D6: D, Diode_SMD:D_SOD-123, symbol Device:D
- added IC2: LM1117IMP-3.3, SamacSys_Parts:SOT230P696X180-4N, symbol SamacSys_Parts:LM1117IMP-3.3
- added J9: USB_C, Connector_USB:USB_C_Receptacle_XKB_U262-16XN-4BVC11, symbol Connector:USB_C_Receptacle_USB2.0
- added JP1, JP2: Jumper_open, Jumper:SolderJumper-2_P1.3mm_Open_RoundedPad1.0x1.5mm, symbol Jumper:SolderJumper_2_Open
- added Q4, Q5: BC847, Package_TO_SOT_SMD:SOT-23, symbol Transistor_BJT:BC847
- added R10, R11: 5k1, Resistor_SMD:R_0402_1005Metric, symbol Device:R
- added R12: 40k, Resistor_SMD:R_0402_1005Metric, symbol Device:R
- added R13: 20k, Resistor_SMD:R_0402_1005Metric, symbol Device:R
- added R21, R22: 10k, Resistor_SMD:R_0402_1005Metric, symbol Device:R
- added U5: CP2102N, Package_DFN_QFN:QFN-24-1EP_4x4mm_P0.5mm_EP2.6x2.6mm, symbol Interface_USB:CP2102N-Axx-xQFN24
- R9: value 10k -> 1k
- gave numbers to parts that had none: 2
Connections:
- net EN_SWITCH is gone; now on net RST: C3.1, R1.2
- net +3.3V: now also C17.2, C5.2, IC2.4 (VOUT_2), U5.5 (VIO), U5.6 (VDD), U5.7 (VREGIN)
- net +5V: now also D6.1 (K), IC2.3 (VIN)
- net CAN_RX: now also U1.13 (IO14); no longer U1.22 (SDI/SD1)
- net CAN_TX: now also U1.16 (IO13); no longer U1.21 (SDO/SD0)
- net GND: now also C17.1, C18.2, C5.1, IC2.1 (ADJ/GND), J9.A1 (GND), J9.A12 (GND), J9.B1 (GND), J9.B12 (GND), J9.S1 (SHIELD), R10.2, R11.1, R13.2, U5.2 (GND), U5.25 (GND)
- net REL3_IN: now also J7.2 (Pin_2); no longer J7.1 (Pin_1)
- net REL3_OUT: now also J7.1 (Pin_1); no longer J7.2 (Pin_2)
- net at R8.2: now also U1.14 (IO12); no longer U1.29 (IO5)
- net at U1.34 (RXD0/IO3): now also JP2.1 (A)
- net at U1.35 (TXD0/IO1): now also JP1.1 (A)
- net BOOT_PIN renamed BOOT
- net BOOT: now also Q5.3 (C)
- net BOOT_SWITCH: no longer names the net of R9.2
- net BOOT_SWITCH: now also U5.9 (~{RST})
- net EN_PIN renamed RST
- net RST: now also Q4.3 (C)
- new net: Q5.1 (B), R22.2
- new net: Q4.1 (B), R21.2
- new net: J9.B5 (CC2), R11.2
- new net: J9.A5 (CC1), R10.1
- new net: R12.2, R13.1, U5.8 (VBUS)
- new net DN: J9.A7 (D-), J9.B7 (D-), U5.4 (D-)
- new net DP: J9.A6 (D+), J9.B6 (D+), U5.3 (D+)
- new net DTR: C18.1, Q5.2 (E), R21.1, U5.23 (~{DTR})
- new net RTS: Q4.2 (E), R22.1, U5.19 (~{RTS})
- new net RXD: JP2.2 (B), U5.21 (TXD)
- new net TXD: JP1.2 (B), U5.20 (RXD)
- new net V_USB: D6.2 (A), J9.A4 (VBUS), J9.A9 (VBUS), J9.B4 (VBUS), J9.B9 (VBUS), R12.1
- no-connect marks 32 -> 43
Other:
- note added: "USB-UART"
- moved on the sheet: C1, C2, C3, C4, R1, R8
